Commit message: Update urdf files

File: src/allegro_hand_controllers/urdf/allegro_hand_description_left_B.urdf (robot description, URDF)
Before this commit: robot allegro_hand_left, 22 links, 21 joints
Links:
- link link_0_0: mass 0.0176 -> 0.0242
- link link_10_0: mass 0.0367 -> 0.0314
- link link_11_0: mass 0.004 -> 0.0275
- link link_11_0_tip: mass 0.0017 -> 0.0018
- link link_12_0: mass 0.0446 -> 0.0416
- link link_13_0: mass 0.0173 -> 0.0224
- link link_14_0: mass 0.03607 -> 0.0315
- link link_15_0: mass 0.0334 -> 0.0545
- link link_15_0_tip: mass 0.0014 -> 0.0015
- link link_1_0: mass 0.086 -> 0.078
- link link_2_0: mass 0.0367 -> 0.0314
- link link_3_0: mass 0.004 -> 0.0275
- link link_3_0_tip: mass 0.0017 -> 0.0018
- link link_4_0: mass 0.0176 -> 0.0242
- link link_5_0: mass 0.086 -> 0.078
- link link_6_0: mass 0.0367 -> 0.0314
- link link_7_0: mass 0.004 -> 0.0275
- link link_7_0_tip: mass 0.0017 -> 0.0018
- link link_8_0: mass 0.0176 -> 0.0242
- link link_9_0: mass 0.086 -> 0.078

File: src/allegro_hand_controllers/urdf/allegro_hand_description_right_B.urdf (robot description, URDF)
Before this commit: robot allegro_hand_right, 22 links, 21 joints
Links:
- link link_0_0: mass 0.0176 -> 0.0242
- link link_10_0: mass 0.0367 -> 0.0314
- link link_11_0: mass 0.004 -> 0.0275
- link link_11_0_tip: mass 0.0017 -> 0.0018
- link link_12_0: mass 0.0446 -> 0.0416
- link link_13_0: mass 0.0173 -> 0.0224
- link link_14_0: mass 0.03607 -> 0.0315
- link link_15_0: mass 0.0334 -> 0.0545
- link link_15_0_tip: mass 0.0014 -> 0.0015
- link link_1_0: mass 0.086 -> 0.078
- link link_2_0: mass 0.0367 -> 0.0314
- link link_3_0: mass 0.004 -> 0.0275
- link link_3_0_tip: mass 0.0017 -> 0.0018
- link link_4_0: mass 0.0176 -> 0.0242
- link link_5_0: mass 0.086 -> 0.078
- link link_6_0: mass 0.0367 -> 0.0314
- link link_7_0: mass 0.004 -> 0.0275
- link link_7_0_tip: mass 0.0017 -> 0.0018
- link link_8_0: mass 0.0176 -> 0.0242
- link link_9_0: mass 0.086 -> 0.078
