Commit message: added allegro and lbr integration

File: allegro_hand_controllers/urdf/allegro_hand_description_right_B.urdf (robot description, URDF)
Before this commit: robot allegro_hand_right, 22 links, 21 joints
Links:
- removed link link_0_0
- removed link link_10_0
- removed link link_11_0
- removed link link_11_0_tip
- removed link link_12_0
- removed link link_13_0
- removed link link_14_0
- removed link link_15_0
- removed link link_15_0_tip
- removed link link_1_0
- removed link link_2_0
- removed link link_3_0
- removed link link_3_0_tip
- removed link link_4_0
- removed link link_5_0
- removed link link_6_0
- removed link link_7_0
- removed link link_7_0_tip
- removed link link_8_0
- removed link link_9_0
- removed link palm_link
Joints:
- removed joint global
- removed joint joint_0_0
- removed joint joint_10_0
- removed joint joint_11_0
- removed joint joint_11_0_tip
- removed joint joint_12_0
- removed joint joint_13_0
- removed joint joint_14_0
- removed joint joint_15_0
- removed joint joint_15_0_tip
- removed joint joint_1_0
- removed joint joint_2_0
- removed joint joint_3_0
- removed joint joint_3_0_tip
- removed joint joint_4_0
- removed joint joint_5_0
- removed joint joint_6_0
- removed joint joint_7_0
- removed joint joint_7_0_tip
- removed joint joint_8_0
- removed joint joint_9_0
